File: videopac_rgb.kicad_pcb (KiCad board)
At the start: 2 copper layers, 80.5 x 41.4 mm, 37 parts, among them J1 RGB Input, J2 DAC Output, Q1 BC558, Q2 BC548, Q3 BC558, Q4 BC548, Q5 BC558, Q6 BC548, Q7 BC548, U1 74HCT32

Commit message: Add additional ground connection.
Parts:
- J2: footprint Connector_PinHeader_2.54mm:PinHeader_1x05_P2.54mm_Horizontal -> Connector_PinHeader_2.54mm:PinHeader_1x06_P2.54mm_Horizontal
- moved J2 1.01 mm to (99.1, 40.1)
- moved Q7 0.66 mm to (94.5, 34.6)
Routing:
- net !CSYNC: track 32.3 -> 27.1 mm
- net +5V: track 123.8 -> 120.8 mm
- net DAC AUDIO: track 32.0 -> 29.4 mm
- net Net-(Q1-Pad2): track 39.1 -> 37.6 mm
- net Net-(D1-Pad2): track 11.5 -> 11.0 mm
Other:
- board text added: "Gnd"
